Commit message: fix:修改urdf路径

File: sdk/src/soarmMoce_sdk/resources/urdf/soarmoce_urdf.urdf (robot description, URDF)
Before this commit: robot soarmoce_urdf, 7 links, 6 joints
Links:
- link base: geometry collision mesh filename=../meshes/base.STL; visual mesh filename=../meshes/base.STL
- link elbow: geometry collision mesh filename=../meshes/elbow.STL; visual mesh filename=../meshes/elbow.STL
- link gripper: geometry collision mesh filename=../meshes/gripper.STL; visual mesh filename=../meshes/gripper.STL
- link shoulder: geometry collision mesh filename=../meshes/shoulder.STL; visual mesh filename=../meshes/shoulder.STL
- link shoulder_lift: geometry collision mesh filename=../meshes/shoulder_lift.STL; visual mesh filename=../meshes/shoulder_lift.STL
- link wrist: geometry collision mesh filename=../meshes/wrist.STL; visual mesh filename=../meshes/wrist.STL
- link wrist_roll: geometry collision mesh filename=../meshes/wrist_roll.STL; visual mesh filename=../meshes/wrist_roll.STL
