Commit message: Add scripts for soarmMoce state diagnosis and URDF zero tuning
- Implemented `soarmmoce_state.py` for reading and diagnosing the current state of the soarmMoce robot, including kinematic analysis and offset hypotheses.
- Created `soarmmoce_urdf_zero_tuner.py` for visual tuning of joint zero offsets in the URDF, allowing interactive adjustments and saving of modified URDF files.
- Added JSON files `soarmmoce_multi_turn_session.json` and `soarmmoce_multi_turn_state.json` to store runtime session and state information for the soarmMoce robot.

File: soarmmoce-real-con/resources/urdf/soarmoce_urdf.urdf (robot description, URDF)
Before this commit: robot soarmoce_urdf, 7 links, 6 joints
Links:
- link base: geometry collision mesh filename=../meshes/base.STL; visual mesh filename=../meshes/base.STL
- link elbow: geometry collision mesh filename=../meshes/elbow.STL; visual mesh filename=../meshes/elbow.STL
- link gripper: geometry collision mesh filename=../meshes/gripper.STL; visual mesh filename=../meshes/gripper.STL
- link shoulder: geometry collision mesh filename=../meshes/shoulder.STL; visual mesh filename=../meshes/shoulder.STL
- link shoulder_lift: geometry collision mesh filename=../meshes/shoulder_lift.STL; visual mesh filename=../meshes/shoulder_lift.STL
- link wrist: geometry collision mesh filename=../meshes/wrist.STL; visual mesh filename=../meshes/wrist.STL
- link wrist_roll: geometry collision mesh filename=../meshes/wrist_roll.STL; visual mesh filename=../meshes/wrist_roll.STL
Joints:
- joint shoulder_lift: origin xyz=0.023908 -0.031327 0.098856 rpy=1.570800 0.000000 1.599500 -> xyz=0.023908 -0.031327 0.098856 rpy=3.141593 1.570793 -3.112889
- joint wrist: origin xyz=-0.152980 0.002177 -0.003775 rpy=0.000000 0.000000 1.570797 -> xyz=-0.152980 0.002177 -0.003775 rpy=0.000000 0.000000 -1.570796
