Commit message: feat: add interactive URDF joint-limit calibrator and enhance zero tuner
- Introduced `soarmmoce_urdf_limit_calibrate.py` for measuring and calibrating URDF joint limits around a user-defined zero pose.
- Updated `soarmmoce_urdf_zero_tuner.py` to clarify its purpose for adjusting joint zero offsets without calibrating limits.
- Implemented JSON output for calibration results, including captured joint limits and relevant metadata.
- Enhanced error handling and path resolution for URDF files and offsets.
- Improved user prompts and logging for better interaction during calibration.

File: skills/soarmmoce-real-con/resources/urdf/1.urdf (robot description, URDF)
Before this commit: robot soarmoce_urdf, 7 links, 6 joints
Links:
- link base: geometry collision mesh filename=../../../../sdk/src/soarmmoce_sdk/resources/meshes/base.STL; visual mesh filename=../../../../sdk/src/soarmmoce_sdk/resources/meshes/base.STL
- link elbow: geometry collision mesh filename=../../../../sdk/src/soarmmoce_sdk/resources/meshes/elbow.STL; visual mesh filename=../../../../sdk/src/soarmmoce_sdk/resources/meshes/elbow.STL
- link gripper: geometry collision mesh filename=../../../../sdk/src/soarmmoce_sdk/resources/meshes/gripper.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; visual mesh filename=../../../../sdk/src/soarmmoce_sdk/resources/meshes/gripper.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
- link shoulder: geometry collision mesh filename=../../../../sdk/src/soarmmoce_sdk/resources/meshes/shoulder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; visual mesh filename=../../../../sdk/src/soarmmoce_sdk/resources/meshes/shoulder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
- link shoulder_lift: geometry collision mesh filename=../../../../sdk/src/soarmmoce_sdk/resources/meshes/shoulder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; visual mesh filename=../../../../sdk/src/soarmmoce_sdk/resources/meshes/shoulder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
- link wrist: geometry collision mesh filename=../../../../sdk/src/soarmmoce_sdk/resources/meshes/wrist.STL; visual mesh filename=../../../../sdk/src/soarmmoce_sdk/resources/meshes/wrist.STL
- link wrist_roll: geometry collision mesh filename=../../../../sdk/src/soarmmoce_sdk/resources/meshes/wrist_ro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; visual mesh filename=../../../../sdk/src/soarmmoce_sdk/resources/meshes/wrist_ro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
Joints:
- joint elbow: limit lower=-1.55342947 upper=1.65752103 effort=0 velocity=0 -> lower=-1.30000000 upper=1.30000000 effort=0 velocity=0
- joint shoulder: limit lower=-1.82543714 upper=2.03252454 effort=0 velocity=0 -> lower=-1.80000000 upper=1.80000000 effort=0 velocity=0
- joint shoulder_lift: limit lower=-1.72124222 upper=1.48738250 effort=0 velocity=0 -> lower=-1.30000000 upper=1.30000000 effort=0 velocity=0; origin xyz=0.023908 -0.031327 0.098856 rpy=1.570800 0.000000 1.599500 -> xyz=0.023908 -0.031327 0.098856 rpy=3.141593 1.570793 -3.112889
- joint wrist: limit lower=-1.59073808 upper=1.52937885 effort=0 velocity=0 -> lower=-1.30000000 upper=1.31000000 effort=0 velocity=0; origin xyz=-0.152980 0.002177 -0.003775 rpy=0.000000 -0.000000 0.000000 -> xyz=-0.152980 0.002177 -0.003775 rpy=0.000000 0.000000 -1.570796
- joint wrist_roll: limit lower=-3.41464123 upper=0.00920388 effort=0 velocity=0 -> lower=-1.30000000 upper=1.30000000 effort=0 velocity=0
