Commit message: Add joint probing and IK testing scripts, enhance SDK with multi-turn handling
- Introduced `soarmmoce_probe_joint_execution.py` for probing joint commands and comparing target vs actual execution.
- Added `soarmmoce_test_xyz_ik.py` for read-only XYZ IK sweeps around the current TCP pose.
- Implemented `soarmmoce_urdf_zero_tuner.py` for visual tuning of joint zero offsets in the URDF.
- Enhanced `soarmmoce_sdk.py` with multi-turn joint handling, including settling logic and improved IK resolution.
- Updated joint model offsets and added user delta to model rotation matrix.
- Improved error handling and diagnostics in IK and movement functions.

File: sdk/src/soarmmoce_sdk/resources/urdf/soarmoce_urdf.urdf (robot description, URDF)
Before this commit: robot soarmoce_urdf, 7 links, 6 joints
Joints:
- joint shoulder_lift: origin xyz=0.023908 -0.031327 0.098856 rpy=1.5708 0 1.5995 -> xyz=0.023908 -0.031327 0.098856 rpy=3.141593 1.570793 -3.112889
- joint wrist: origin xyz=-0.15298 0.0021767 -0.003775 rpy=0 0 0 -> xyz=-0.152980 0.002177 -0.003775 rpy=0.000000 0.000000 -1.570796

Commit message: Refactor calibration and URDF handling for single-turn joints
- Updated soarmmoce.json to adjust homing offsets, range limits, and added zero_present_raw for several joints.
- Enhanced urdf_calibrate.py to support new zero_present_raw parameter and validate calibration ranges.
- Implemented logic to write updated joint limits to URDF in urdf_calibrate.py.
- Modified urdf_zero_tuner.py to shift existing joint limits when adjusting joint origins.
- Improved real_arm.py to include zero_raw in joint specifications and validate joint goals against calibrated ranges.
- Adjusted URDF definitions in soarmoce_urdf.urdf to reflect new joint limits and orientations.
- Added max_joint_delta_rad parameter to move functions for better IK control.

File: sdk/src/soarmmoce_sdk/resources/urdf/soarmoce_urdf.urdf (robot description, URDF)
Before this commit: robot soarmoce_urdf, 7 links, 6 joints
Joints:
- joint elbow: limit lower=-1.55342947 upper=1.65752103 effort=0 velocity=0 -> lower=-3.12422580 upper=0.08672470 effort=0 velocity=0; origin xyz=-0.036111 0.12717 0.0005 rpy=0 0 0 -> xyz=-0.036111 0.127170 0.000500 rpy=0.000000 -0.000000 1.570796
- joint shoulder: limit lower=-1.82543714 upper=2.03252454 effort=0 velocity=0 -> lower=-1.79322354 upper=1.83310704 effort=0 velocity=0
- joint shoulder_lift: limit lower=-1.72124222 upper=1.48738250 effort=0 velocity=0 -> lower=-0.15044589 upper=3.05817883 effort=0 velocity=0; origin xyz=0.023908 -0.031327 0.098856 rpy=1.570800 0.000000 1.599500 -> xyz=0.023908 -0.031327 0.098856 rpy=3.141593 1.570793 -3.112889
- joint wrist: limit lower=-1.59073808 upper=1.52937885 effort=0 velocity=0 -> lower=-2.77190328 upper=0.36815539 effort=0 velocity=0; origin xyz=-0.152980 0.002177 -0.003775 rpy=0.000000 -0.000000 0.000000 -> xyz=-0.152980 0.002177 -0.003775 rpy=0.000000 -0.000000 -1.570796
